File: DRC-CanTester.kicad_pcb (KiCad board)
At the start: 2 copper layers, 60 x 60 mm, 47 parts, among them J1 CAN, J2 STLINK, J3 USB_C, SW1 MODE, SW2 BUS-OFF_RESET, SW3 TEST, SW4 RESET, U1 RT9080-33GJ5, U2 STM32F303K8Tx, U3 CH340E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

Commit message: シルクを修正
Other:
- board text added: "DRC-CanTester v0.1.0"
- board text removed: "DRC-CanTester v0.0.1"
Changed lines of the file:
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@@
 		)
 	)
-	(gr_text "DRC-CanTester v0.0.1"
+	(gr_text "DRC-CanTester v0.1.0"
 		(at 187.15 65.55 0)
 		(layer "B.SilkS")
@@
 			(justify left bottom mirror)
 		)
-		(render_cache "DRC-CanTester v0.0.1" 0
+		(render_cache "DRC-CanTester v0.1.0" 0
 			(polygon
 				(pts
@@
 			(polygon
 				(pts
-					(xy 149.972723 62.009349) (xy 150.066014 62.026335) (xy 150.23632 62.091963) (xy 150.388823 62.19977)
-					(xy 150.525265 62.352871) (xy 150.644478 62.556589) (xy 150.742325 62.816132) (xy 150.812204 63.133654)
-					(xy 150.846194 63.504828) (xy 150.848246 63.6262) (xy 150.842174 63.857523) (xy 150.823114 64.079674)
-					(xy 150.795059 64.263024) (xy 150.755439 64.435718) (xy 150.710493 64.577103) (xy 150.655447 64.707769)
-					(xy 150.597443 64.814202) (xy 150.530583 64.910361) (xy 150.46166 64.988287) (xy 150.384767 65.056377)
-					(xy 150.30517 65.110723) (xy 150.218059 65.155352) (xy 150.126231 65.188845) (xy 150.02689 65.212253)
-					(xy 149.844408 65.227578) (xy 149.743534 65.221803) (xy 149.64864 65.204823) (xy 149.476842 65.139524)
-					(xy 149.324458 65.032768) (xy 149.189179 64.881643) (xy 149.071597 64.680661) (xy 148.975275 64.423904)
-					(xy 148.906301 64.107807) (xy 148.872301 63.734672) (xy 148.87028 63.617773) (xy 149.37821 63.617773)
-					(xy 149.384314 63.854129) (xy 149.4036 64.079115) (xy 149.430948 64.253826) (xy 149.469415 64.411822)
-					(xy 149.509903 64.526224) (xy 149.558932 64.624474) (xy 149.606249 64.691934) (xy 149.659995 64.745604)
-					(xy 149.711496 64.779749) (xy 149.768106 64.802013) (xy 149.844408 64.811938) (xy 149.912819 64.80618)
-					(xy 149.975093 64.789325) (xy 150.081677 64.725336) (xy 150.171842 64.617345) (xy 150.247684 64.453753)
-					(xy 150.306309 64.217383) (xy 150.341549 63.887888) (xy 150.348342 63.621987) (xy 150.342355 63.392938)
-					(xy 150.323889 63.176244) (xy 150.296785 63.000117) (xy 150.258966 62.840804) (xy 150.21826 62.721764)
-					(xy 150.169222 62.619232) (xy 150.121489 62.547524) (xy 150.067508 62.490064) (xy 150.015984 62.452987)
-					(xy 149.959596 62.428097) (xy 149.8739 62.415183) (xy 149.805499 62.420947) (xy 149.743362 62.437851)
-					(xy 149.637862 62.501796) (xy 149.54924 62.609678) (xy 149.475128 62.773675) (xy 149.418215 63.01246)
-					(xy 149.384403 63.350061) (xy 149.37821 63.617773) (xy 148.87028 63.617773) (xy 148.870062 63.605134)
-					(xy 148.876047 63.388332) (xy 148.89449 63.178935) (xy 148.922583 62.997503) (xy 148.962062 62.8258)
-					(xy 149.007683 62.681288) (xy 149.063329 62.547283) (xy 149.122349 62.436637) (xy 149.190112 62.33645)
-					(xy 149.259811 62.254943) (xy 149.337249 62.183607) (xy 149.416716 62.126807) (xy 149.503297 62.080045)
-					(xy 149.593413 62.045078) (xy 149.69043 62.020418) (xy 149.8739 62.003572)
+					(xy 149.201805 65.16896) (xy 149.17104 65.163093) (xy 149.14947 65.14547) (xy 149.13879 65.106128)
+					(xy 149.13879 64.887592) (xy 149.145614 64.840903) (xy 149.16182 64.824454) (xy 149.193379 64.816334)
+					(xy 149.407864 64.791468) (xy 149.466585 64.769561) (xy 149.501758 64.736287) (xy 149.524383 64.660385)
+					(xy 149.529518 64.589188) (xy 149.538816 64.337842) (xy 149.541974 64.206704) (xy 149.535305 63.220647)
+					(xy 149.512063 62.44354) (xy 149.491599 62.151034) (xy 149.487386 62.083806) (xy 149.493407 62.040345)
+					(xy 149.512106 62.018188) (xy 149.541974 62.012365) (xy 149.584106 62.016578) (xy 149.824917 62.052667)
+					(xy 150.029754 62.070659) (xy 150.218283 62.07538) (xy 150.297967 62.07538) (xy 150.322743 62.081567)
+					(xy 150.34149 62.101431) (xy 150.348342 62.134181) (xy 150.35038 62.25122) (xy 150.352555 62.377814)
+					(xy 150.344152 62.433913) (xy 150.327748 62.445614) (xy 150.297967 62.449071) (xy 150.071874 62.457238)
+					(xy 150.024099 62.470039) (xy 150.004016 62.490957) (xy 149.999747 62.524909) (xy 149.991503 63.050458)
+					(xy 150.009246 64.140683) (xy 150.029239 64.593401) (xy 150.045007 64.707837) (xy 150.074266 64.761724)
+					(xy 150.138415 64.786842) (xy 150.27753 64.806101) (xy 150.40293 64.812121) (xy 150.425679 64.824478)
+					(xy 150.445183 64.851872) (xy 150.449275 64.875136) (xy 150.446346 65.024908) (xy 150.445062 65.080849)
+					(xy 150.439041 65.128792) (xy 150.420342 65.159131) (xy 150.390474 65.16896) (xy 150.382048 65.16896)
+					(xy 149.781393 65.156503) (xy 149.210232 65.16896)
 				)
 			)
@@
 			(polygon
 				(pts
-					(xy 145.719879 65.16896) (xy 145.689114 65.163093) (xy 145.667544 65.14547) (xy 145.656864 65.106128)
-					(xy 145.656864 64.887592) (xy 145.663688 64.840903) (xy 145.679894 64.824454) (xy 145.711453 64.816334)
-					(xy 145.925938 64.791468) (xy 145.984659 64.769561) (xy 146.019832 64.736287) (xy 146.042457 64.660385)
-					(xy 146.047592 64.589188) (xy 146.05689 64.337842) (xy 146.060048 64.206704) (xy 146.053379 63.220647)
-					(xy 146.030137 62.44354) (xy 146.009673 62.151034) (xy 146.00546 62.083806) (xy 146.011481 62.040345)
-					(xy 146.03018 62.018188) (xy 146.060048 62.012365) (xy 146.10218 62.016578) (xy 146.342991 62.052667)
-					(xy 146.547828 62.070659) (xy 146.736357 62.07538) (xy 146.816041 62.07538) (xy 146.840817 62.081567)
-					(xy 146.859564 62.101431) (xy 146.866416 62.134181) (xy 146.868454 62.25122) (xy 146.870629 62.377814)
-					(xy 146.862226 62.433913) (xy 146.845822 62.445614) (xy 146.816041 62.449071) (xy 146.589948 62.457238)
-					(xy 146.542173 62.470039) (xy 146.52209 62.490957) (xy 146.517821 62.524909) (xy 146.509577 63.050458)
-					(xy 146.52732 64.140683) (xy 146.547313 64.593401) (xy 146.563081 64.707837) (xy 146.59234 64.761724)
-					(xy 146.656489 64.786842) (xy 146.795604 64.806101) (xy 146.921004 64.812121) (xy 146.943753 64.824478)
-					(xy 146.963257 64.851872) (xy 146.967349 64.875136) (xy 146.96442 65.024908) (xy 146.963136 65.080849)
-					(xy 146.957115 65.128792) (xy 146.938416 65.159131) (xy 146.908548 65.16896) (xy 146.900122 65.16896)
-					(xy 146.299467 65.156503) (xy 145.728306 65.16896)
-				)
-			)
+					(xy 146.490797 62.009349) (xy 146.584088 62.026335) (xy 146.754394 62.091963) (xy 146.906897 62.19977)
+					(xy 147.043339 62.352871) (xy 147.162552 62.556589) (xy 147.260399 62.816132) (xy 147.330278 63.133654)
+					(xy 147.364268 63.504828) (xy 147.36632 63.6262) (xy 147.360248 63.857523) (xy 147.341188 64.079674)
+					(xy 147.313133 64.263024) (xy 147.273513 64.435718) (xy 147.228567 64.577103) (xy 147.173521 64.707769)
+					(xy 147.115517 64.814202) (xy 147.048656 64.910361) (xy 146.979734 64.988287) (xy 146.902841 65.056377)
+					(xy 146.823244 65.110723) (xy 146.736133 65.155352) (xy 146.644305 65.188845) (xy 146.544964 65.212253)
+					(xy 146.362482 65.227578) (xy 146.261608 65.221803) (xy 146.166714 65.204823) (xy 145.994916 65.139524)
+					(xy 145.842532 65.032768) (xy 145.707253 64.881643) (xy 145.589671 64.680661) (xy 145.493349 64.423904)
+					(xy 145.424375 64.107807) (xy 145.390375 63.734672) (xy 145.388354 63.617773) (xy 145.896284 63.617773)
+					(xy 145.902388 63.854129) (xy 145.921674 64.079115) (xy 145.949022 64.253826) (xy 145.987489 64.411822)
+					(xy 146.027977 64.526224) (xy 146.077006 64.624474) (xy 146.124323 64.691934) (xy 146.178069 64.745604)
+					(xy 146.229569 64.779749) (xy 146.28618 64.802013) (xy 146.362482 64.811938) (xy 146.430893 64.80618)
+					(xy 146.493167 64.789325) (xy 146.599751 64.725336) (xy 146.689916 64.617345) (xy 146.765758 64.453753)
+					(xy 146.824383 64.217383) (xy 146.859623 63.887888) (xy 146.866416 63.621987) (xy 146.860429 63.392938)
+					(xy 146.841963 63.176244) (xy 146.814859 63.000117) (xy 146.77704 62.840804) (xy 146.736334 62.721764)
+					(xy 146.687296 62.619232) (xy 146.639563 62.547524) (xy 146.585582 62.490064) (xy 146.534058 62.452987)
+					(xy 146.47767 62.428097) (xy 146.391974 62.415183) (xy 146.323573 62.420947) (xy 146.261436 62.437851)
+					(xy 146.155936 62.501796) (xy 146.067314 62.609678) (xy 145.993202 62.773675) (xy 145.936289 63.01246)
+					(xy 145.902477 63.350061) (xy 145.896284 63.617773) (xy 145.388354 63.617773) (xy 145.388136 63.605134)
+					(xy 145.394121 63.388332) (xy 145.412564 63.178935) (xy 145.440657 62.997503) (xy 145.480136 62.8258)
+					(xy 145.525757 62.681288) (xy 145.581402 62.547283) (xy 145.640423 62.436637) (xy 145.708186 62.33645)
+					(xy 145.777885 62.254943) (xy 145.855323 62.183607) (xy 145.93479 62.126807) (xy 146.021371 62.080045)
+					(xy 146.111487 62.045078) (xy 146.208504 62.020418) (xy 146.391974 62.003572)
+				)
+			)
